Commit message: Added Core URDF

File: description/robot_core.xacro (robot description, xacro)
@@ -37,4 +37,7 @@
             </geometry>
         </collision>
+        <xacro:inertial_box mass="0.5" x="0.3" y="0.3" z="0.3">
+            <origin xyz="0.15 0.0 0.075" rpy="0.0 0.0 0.0"/>
+        </xacro:inertial_box>
     </link>
     <!-- Left Wheel Link -->
@@ -57,4 +60,7 @@
             </geometry>
         </collision>
+        <xacro:inertial_cylinder mass="0.1" length="0.04">
+            <origin xyz="0.0 0.0 0.0" rpy="0.0 0.0 0.0"/>
+        </xacro:inertial_cylinder>
     </link>
 <!-- Right Wheel Link -->
@@ -77,4 +83,7 @@
             </geometry>
         </collision>
+        <xacro:inertial_cylinder mass="0.1" length="0.04">
+            <origin xyz="0.0 0.0 0.0" rpy="0.0 0.0 0.0"/>
+        </xacro:inertial_cylinder>
     </link>
 <!-- Caster Wheel Link -->
@@ -96,4 +105,7 @@
             </geometry>
         </collision>
+        <xacro:inertial_sphere mass="0.1" radius="0.05">
+            <origin xyz="0.0 0.0 0.0" rpy="0.0 0.0 0.0"/>
+        </xacro:inertial_sphere>
     </link>
 </robot>

Commit message: Added Gazebo Tags

File: description/robot_core.xacro (robot description, xacro)
@@ -41,4 +41,7 @@
         </xacro:inertial_box>
     </link>
+    <gazebo reference="chassis_link">
+    <material>Gazebo/White</material>
+    </gazebo>
     <!-- Left Wheel Link -->
     <joint name="left_wheel_joint" type="continuous">
@@ -64,4 +67,7 @@
         </xacro:inertial_cylinder>
     </link>
+    <gazebo reference="left_wheel_link">
+        <material>Gazebo/Blue</material>
+    </gazebo>
 <!-- Right Wheel Link -->
     <joint name="right_wheel_joint" type="continuous">
@@ -83,8 +89,11 @@
             </geometry>
         </collision>
-        <xacro:inertial_cylinder mass="0.1" length="0.04">
+        <xacro:inertial_cylinder mass="0.1" length="0.04" radius="0.05">
             <origin xyz="0.0 0.0 0.0" rpy="0.0 0.0 0.0"/>
         </xacro:inertial_cylinder>
     </link>
+    <gazebo reference="right_wheel_link">
+        <material>Gazebo/Blue</material>
+    </gazebo>
 <!-- Caster Wheel Link -->
     <joint name="caster_joint" type="fixed">
@@ -109,3 +118,6 @@
         </xacro:inertial_sphere>
     </link>
+    <gazebo reference="caster_wheel_link">
+        <material>Gazebo/Black</material>
+    </gazebo>
 </robot>
